File: Macro Pad/Macro Pad.kicad_pcb (KiCad board)
At the start: 2 copper layers, 118 x 92.5 mm, 17 parts, among them SW1 SW_Push, SW10 SW_Push, SW11 SW_Push, SW12 SW_Push, SW2 SW_Push, SW3 SW_Push, SW4 SW_Push, SW5 SW_Push, SW6 SW_Push, SW7 SW_Push, SW8 SW_Push, SW9 SW_Push

Commit message: Completed PCB
Parts:
- S1: value SWITCH -> sdpt; footprint Button_Switch_THT:SW_Slide-03_Wuerth-WS-SLTV_10x2.5x6.4_P2.54mm -> spdt:SW_ATE1D-2M3-10-Z
- moved S1 0.50 mm to (171.0, 103.0), turned to -90 degrees
Connections:
- S1 pad 1: 5V -> Net-(Ch1-OUT+)
- S1 pad 2: Net-(Ch1-OUT+) -> 5V
Routing:
- net GND: track 573.1 -> 596.4 mm, vias 0 -> 1
- net 5V: track 142.0 -> 147.3 mm
- net Net-(MCU1-D19): track 107.3 -> 108.2 mm
- net Net-(MCU1-D21): track 147.9 -> 148.8 mm
- net unconnected-(MCU1-D23-Pad15): vias 1 -> 0
- added copper zone on B.Cu, net GND
- added copper zone on F.Cu, net GND
Other:
- board text added: "D12, SW5"
- board text added: "D13, SW1"
- board text added: "D14, SW8"
- board text added: "D15, SW11"
- board text added: "D18, SW12"
- board text added: "D21"
- board text added: "D22"
- board text added: "D23"
- board text added: "D25, SW6"
- board text added: "D26, SW2"
- board text added: "D27, B, CLK"
- board text added: "D32, A, Data"
- board text added: "D33, SW9"
- board text added: "D34, SW7"
- board text added: "D35, SW10"
- board text added: "EN"
- board text added: "ESP32 Based Macro Pad MODES: Bluetooth ONLY Original Creator: theNeonTerminal https://github.com/theNeonTerminal/Macro-Pad"
- board text added: "GND"
- board text added: "SCL"
- board text added: "SDA"
- board text added: "USB-C"
- board text added: "VCC"
- board text added: "VN(39), SW4"
- board text added: "VP(36), SW3"
