File: Macro Pad/Macro Pad.kicad_sch (KiCad schematic)
At the start: 17 parts, among them SW1 SW_Push, SW10 SW_Push, SW11 SW_Push, SW12 SW_Push, SW2 SW_Push, SW3 SW_Push, SW4 SW_Push, SW5 SW_Push, SW6 SW_Push, SW7 SW_Push, SW8 SW_Push, SW9 SW_Push

Commit message: Completed PCB
Parts:
- removed S1: SWITCH, Button_Switch_THT:SW_Slide-03_Wuerth-WS-SLTV_10x2.5x6.4_P2.54mm, symbol Simulation_SPICE:SWITCH
- added S1: sdpt, spdt:SW_ATE1D-2M3-10-Z, symbol spdt:ATE1D-2M3-10-Z
Connections:
- net at Ch1.OUT_P (OUT+): now also S1.1
- net +5V renamed 5V
- net 5V: now also S1.2
- no-connect marks 0 -> 15

Commit message: Project Completed (mostly)
Parts:
- renumbered OLED1 to OLED
Changed lines of the file:
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@@
 		(in_pos_files yes)
 		(dnp no)
-		(property "Reference" "OLED1"
+		(property "Reference" "OLED"
 			(at 73.914 105.918 90)
 			(show_name no)
@@
 			(project "Macro Pad"
 				(path "/09e6d6cb-ab99-4d7a-8962-ceabe82c0aef"
-					(reference "OLED1")
+					(reference "OLED")
 					(unit 1)
 				)
